File: LS.kicad_sch (KiCad schematic)
At the start: 12 parts, among them U3 VNLD5160TR-E, U4 VNLD5160TR-E

Commit message: Rev G
Connections:
- net +12V_RAW renamed +12V
Changed lines of the file:
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@@
+    )
+  )
+  (symbol (lib_id "power:+12V") (at 142.24 20.32 0) (unit 1)
+    (in_bom yes) (on_board yes) (dnp no)
+    (property "Reference" "#PWR06" (at 142.24 24.13 0)
+      (effects (font (size 1.27 1.27)) hide)
+    )
+    (property "Value" "+12V" (at 142.24 16.51 0)
+      (effects (font (size 1.27 1.27)))
+    )
+    (property "Footprint" "" (at 142.24 20.32 0)
+      (effects (font (size 1.27 1.27)) hide)
+    )
+    (property "Datasheet" "" (at 142.24 20.32 0)
+      (effects (font (size 1.27 1.27)) hide)
+    )
+    (pin "1")
+    (instances
+      (project "PROLT"
+        (path "/b8382448-02ab-4b6d-b574-50f724fc5555/4d1d140e-577f-4c68-bab8-9a91e78a044c"
+          (reference "#PWR06") (unit 1)
+        )
+      )
     )
   )
@@
     )
   )
-  (symbol (lib_id "misc:+12V_RAW") (at 142.24 45.72 0) (unit 1)
-    (in_bom yes) (on_board yes) (dnp no)
-    (property "Reference" "#PWR016" (at 142.24 49.53 0)
-      (effects (font (size 1.27 1.27)) hide)
-    )
-    (property "Value" "+12V_RAW" (at 142.24 41.91 0)
+  (symbol (lib_id "power:GND") (at 58.42 93.98 0) (unit 1)
+    (in_bom yes) (on_board yes) (dnp no)
+    (property "Reference" "#PWR070" (at 58.42 100.33 0)
+      (effects (font (size 1.27 1.27)) hide)
+    )
+    (property "Value" "GND" (at 58.42 97.79 0)
+      (effects (font (size 1.27 1.27)))
+    )
+    (property "Footprint" "" (at 58.42 93.98 0)
+      (effects (font (size 1.27 1.27)) hide)
+    )
+    (property "Datasheet" "" (at 58.42 93.98 0)
+      (effects (font (size 1.27 1.27)) hide)
+    )
+    (pin "1")
+    (instances
+      (project "PROLT"
+        (path "/b8382448-02ab-4b6d-b574-50f724fc5555/4d1d140e-577f-4c68-bab8-9a91e78a044c"
+          (reference "#PWR070") (unit 1)
+        )
+      )
+    )
+  )
+  (symbol (lib_id "power:+12V") (at 142.24 45.72 0) (unit 1)
+    (in_bom yes) (on_board yes) (dnp no)
+    (property "Reference" "#PWR015" (at 142.24 49.53 0)
+      (effects (font (size 1.27 1.27)) hide)
+    )
+    (property "Value" "+12V" (at 142.24 41.91 0)
       (effects (font (size 1.27 1.27)))
     )
@@
       (project "PROLT"
         (path "/b8382448-02ab-4b6d-b574-50f724fc5555/4d1d140e-577f-4c68-bab8-9a91e78a044c"
-          (reference "#PWR016") (unit 1)
-        )
-      )
-    )
-  )
-  (symbol (lib_id "power:GND") (at 58.42 93.98 0) (unit 1)
-    (in_bom yes) (on_board yes) (dnp no)
-    (property "Reference" "#PWR070" (at 58.42 100.33 0)
-      (effects (font (size 1.27 1.27)) hide)
-    )
-    (property "Value" "GND" (at 58.42 97.79 0)
-      (effects (font (size 1.27 1.27)))
-    )
-    (property "Footprint" "" (at 58.42 93.98 0)
-      (effects (font (size 1.27 1.27)) hide)
-    )
-    (property "Datasheet" "" (at 58.42 93.98 0)
-      (effects (font (size 1.27 1.27)) hide)
-    )
-    (pin "1")
-    (instances
-      (project "PROLT"
-        (path "/b8382448-02ab-4b6d-b574-50f724fc5555/4d1d140e-577f-4c68-bab8-9a91e78a044c"
-          (reference "#PWR070") (unit 1)
+          (reference "#PWR015") (unit 1)
         )
       )
@@
         )
       )
-    )
-  )
-  (symbol (lib_id "misc:+12V_RAW") (at 142.24 20.32 0) (unit 1)
-    (in_bom yes) (on_board yes) (dnp no)
-    (property "Reference" "#PWR015" (at 142.24 24.13 0)
-      (effects (font (size 1.27 1.27)) hide)
-    )
-    (property "Value" "+12V_RAW" (at 142.24 16.51 0)
-      (effects (font (size 1.27 1.27)))
-    )
-    (property "Footprint" "" (at 142.24 20.32 0)
-      (effects (font (size 1.27 1.27)) hide)
-    )
-    (property "Datasheet" "" (at 142.24 20.32 0)
-      (effects (font (size 1.27 1.27)) hide)
-    )
-    (pin "1")
-    (instances
-      (project "PROLT"
-        (path "/b8382448-02ab-4b6d-b574-50f724fc5555/4d1d140e-577f-4c68-bab8-9a91e78a044c"
-          (reference "#PWR015") (unit 1)
-        )
-      )
