File: PROLT.kicad_pcb (KiCad board)
At the start: 4 copper layers, 80 x 80 mm, 93 parts, among them IC1 BTS4175SGA, IC2 IFX9201SGAUMA1, IC3 IFX9201SGAUMA1, J1 64334-0100, J2 USB, M1 Module:mega-mcu100/0.3, M2 Module-vr-max9924-0.1, M3 Module-power_12and5V-0.2, U1 VNLD5160TR-E, U2 VNLD5160TR-E, U3 VNLD5160TR-E, U4 VNLD5160TR-E

Commit message: Rev G
Parts:
- added U5: BTS3046SDRATMA1, easyeda2kicad:PG-TO252-3_L6.5-W6.2-P4.57-LS10.0-BR-CW-1, F.Cu at (145.9, 86.6)
- added U6: BTS3046SDRATMA1, easyeda2kicad:PG-TO252-3_L6.5-W6.2-P4.57-LS10.0-BR-CW-1, F.Cu at (167.0, 86.7)
- C1, D1, D2, IC1, JP1, JP2, R10, R21, R22, R23, R24, R25, R26, R5, R6, R7, R8, R9, U3, U4: moved to B.Cu
- R1, R17, R18, R19, R2, R20, R3, R4: value 4.7k -> 10k
- U1, U2: value VNLD5160TR-E -> BTS3046SDRATMA1; footprint Package_SO:SOIC-8_3.9x4.9mm_P1.27mm -> easyeda2kicad:PG-TO252-3_L6.5-W6.2-P4.57-LS10.0-BR-CW-1
- moved JP1 20.8 mm to (173.5, 60.6)
- moved D2 19.0 mm to (132.2, 60.6), turned to 0 degrees
- moved D1 18.0 mm to (132.2, 62.9), turned to 0 degrees
- moved R9 17.8 mm to (161.5, 86.7)
- moved JP2 17.7 mm to (173.5, 64.3)
- moved R21 15.4 mm to (160.3, 86.7)
- moved R26 14.5 mm to (150.2, 86.7)
- moved U4 14.1 mm to (159.6, 80.7)
- moved R10 13.0 mm to (159.0, 86.7)
- moved R24 12.0 mm to (151.5, 86.7)
- moved U3 11.9 mm to (152.1, 80.7)
- moved R22 10.7 mm to (157.8, 86.7)
- moved R20 10.2 mm to (168.8, 92.3), turned to 0 degrees
- moved R25 9.66 mm to (152.8, 86.7)
- moved R7 8.11 mm to (165.1, 86.7)
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Connections:
- D1 pad 1: +12V_RAW -> +12V
- D2 pad 1: +12V_RAW -> +12V
- R1 pad 1: GND -> Net-(U1-IN)
- R1 pad 2: /INJ1_IN -> /INJ2_IN
- R17 pad 1: GND -> Net-(U2-IN)
- R18 pad 1: GND -> Net-(U6-IN)
- R19 pad 1: Net-(U2-IN1) -> /INJ3_IN
- R19 pad 2: /INJ3_IN -> GND
- R2 pad 1: GND -> /INJ1_IN
- R2 pad 2: /INJ2_IN -> GND
- R20 pad 1: Net-(U2-IN2) -> /INJ4_IN
- R20 pad 2: /INJ4_IN -> GND
- R3 pad 1: Net-(U1-IN1) -> Net-(U5-IN)
- R4 pad 1: Net-(U1-IN2) -> /INJ2_IN
- R4 pad 2: /INJ2_IN -> GND
- U1 pad 1: Net-(U1-IN1) -> Net-(U1-IN)
- U1 pad 2: unconnected-(U1-STATUS1-Pad2) -> /INJ2_OUT
- U1 pad 3: Net-(U1-IN2) -> GND
- U2 pad 1: Net-(U2-IN1) -> Net-(U2-IN)
- U2 pad 2: unconnected-(U2-STATUS1-Pad2) -> /INJ3_OUT
- U2 pad 3: Net-(U2-IN2) -> GND
Routing:
- net /OUT_4: track 3.70 -> 33.3 mm
- net /OUT_1: track 20.0 -> 49.3 mm
- net /OUT_3: track 7.28 -> 32.5 mm
- net +12V: track 95.1 -> 112.3 mm
- net /LowSide Outputs/IN_4: track 12.4 -> 24.1 mm, vias 0 -> 2
- net /LS1: track 11.3 -> 22.7 mm, vias 0 -> 2
- net Net-(JP2-C): track 31.4 -> 42.5 mm
- net Net-(JP1-C): track 15.9 -> 25.6 mm
- net /HS: track 17.4 -> 26.9 mm, vias 2 -> 1
- net +3.3V: track 189.2 -> 179.7 mm
- net /LS2: track 17.1 -> 25.9 mm
- net /IGN3_OUT: track 19.1 -> 27.9 mm, vias 2 -> 3
- net /OUT_2: track 34.0 -> 42.8 mm
- net /INJ4_IN: track 10.5 -> 18.5 mm
- net /INJ4_OUT: track 13.6 -> 21.5 mm
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- added copper zone on F.Cu, net /INJ1_OUT
- added copper zone on F.Cu, net /INJ2_OUT
- added copper zone on F.Cu, net /INJ3_OUT
- added copper zone on F.Cu, net /INJ4_OUT
Other:
- board text added: "<<< DIN 3 / OUT 4 >>>"
- board text added: "<<< IGN 3 / OUT 3 >>>"
- board text added: "PROLT REV.G"
- board text removed: "<<< OUT 3 / ING 3 >>>"
- board text removed: "<<< OUT 4 / DIN 3 >>>"
- board text removed: "PROLT REV.E"
